File: Hardware/Flight Controller/Misc.kicad_sch (KiCad schematic)
At the start: 61 parts, among them CN1 1.0-8P WT, CN2 1.0-6P WT, CN3 1.0-5P WT, CN4 1.0-4P WT, J1 Conn_01x04_Pin, J2 Conn_01x08_Pin, J3 Conn_01x06_Pin, J4 Conn_01x05_Pin, J5 Conn_01x04_Pin, J6 Conn_01x04_Pin, J7 Conn_01x04_Pin, J8 Conn_01x03_Pin, Q1 MMBT2222A, SW1_BOOT1 TS-1088-AR02016, SW1_RST1 TS-1088-AR02016, U6 KLJ-9650-5Y, X2 X322525MOB4SI, X3 Q13FC1350000200

Commit message: Done?
Parts:
- C32, C33: value 20pF -> 18pf
- C34, C35: value 6.8pF -> 18pf
- X3: footprint lcsc:FC-135R_L3.2-W1.5 -> SMD3215-2P:CHIP_NX3215S_NDK
Other:
- moved on the sheet: C33
