File: Hardware/Flight Controller/Flight Controller.kicad_pcb (KiCad board)
At the start: 2 copper layers, 51.3 x 55.3 mm, 123 parts, among them CN1 1.0-8P WT, CN2 1.0-6P WT, CN3 1.0-5P WT, CN4 1.0-4P WT, J1 Conn_01x04_Pin, J2 Conn_01x08_Pin, J3 Conn_01x06_Pin, J4 Conn_01x05_Pin, J5 Conn_01x04_Pin, J6 Conn_01x04_Pin, J7 Conn_01x04_Pin, J8 Conn_01x03_Pin, Q1 MMBT2222A, SW1_BOOT1 TS-1088-AR02016, SW1_RST1 TS-1088-AR02016, U1 STM32F722RETx, U2 AT7456E, U3 LMR51430, U4 TPS63070RNMR, U5 TPS63070RNMR, U6 KLJ-9650-5Y, U8 ICM-45686, U9 BMP280, X1 27Mhz, X2 X322525MOB4SI, X3 Q13FC1350000200

Commit message: Done?
Parts:
- C34, C35: value 6.8pF -> 12pf
- X3: footprint lcsc:FC-135R_L3.2-W1.5 -> SMD3215-2P:CHIP_NX3215S_NDK
- moved C35 0.59 mm to (140.8, 79.2)
- moved C34 0.25 mm to (142.8, 76.2), turned to 180 degrees
Routing:
- net BUZZER: track 36.2 -> 34.4 mm
- net +3.3V: track 156.2 -> 155.4 mm
- net GND: track 90.2 -> 89.4 mm, vias 467 -> 466
- net M_4: track 29.7 -> 29.1 mm
- net LSE_CLK_IN: track 7.46 -> 7.98 mm
- net Video_In: track 59.2 -> 58.7 mm
Other:
- board text added: "Design By Ari H"

Commit message: Lock In Twin
Parts:
- C32, C33: value 20pF -> 18pf
- C34, C35: value 12pf -> 18pf
